Commit message: added robot

File: robot.urdf (robot description, URDF)
Before this commit: robot robot, 4 links, 3 joints
Links:
- added link box, mass 0.5; collision box size=0.4 0.3 0.1; visual box size=0.4 0.3 0.1
Joints:
- added joint joint4: type fixed, parent link3, child box, origin xyz=0.5 0 0 rpy=0 0 0
- joint joint1: limit lower=0.0 upper=3.14 -> lower=0.0 upper=3.14 effort=100.0 velocity=2.0
- joint joint2: limit lower=-1.57 upper=1.57 -> lower=-1.57 upper=1.57 effort=100.0 velocity=2.0; origin xyz=0 0 0 rpy=0 0 0 -> xyz=0.5 0 0 rpy=0 0 0
- joint joint3: limit lower=-1.57 upper=1.57 -> lower=-1.57 upper=1.57 effort=100.0 velocity=2.0; origin xyz=0 0 0 rpy=0 0 0 -> xyz=0.5 0 0 rpy=0 0 0; parent link3 -> link2
